File: 61key.kicad_pcb (KiCad board)
At the start: 2 copper layers, 134 parts, among them J1 105450-0101, SW1 SW_SPST, SW10 SW_SPST, SW11 SW_SPST, SW12 SW_SPST, SW13 SW_SPST, SW14 SW_SPST, SW15 SW_SPST, SW16 SW_SPST, SW17 SW_SPST, SW18 SW_SPST, SW19 SW_SPST, SW2 SW_SPST, SW20 SW_SPST, SW21 SW_SPST, SW22 SW_SPST, SW23 SW_SPST, SW24 SW_SPST, SW25 SW_SPST, SW26 SW_SPST, SW27 SW_SPST, SW28 SW_SPST, SW29 SW_SPST, SW3 SW_SPST, SW30 SW_SPST, SW31 SW_SPST, SW32 SW_SPST, SW33 SW_SPST, SW34 SW_SPST, SW35 SW_SPST, SW36 SW_SPST, SW37 SW_SPST, SW38 SW_SPST, SW39 SW_SPST, SW4 SW_SPST, SW40 SW_SPST, SW41 SW_SPST, SW42 SW_SPST, SW43 SW_SPST, SW44 SW_SPST, SW45 SW_SPST, SW46 SW_SPST, SW47 SW_SPST, SW48 SW_SPST, SW49 SW_SPST, SW5 SW_SPST, SW50 SW_SPST, SW51 SW_SPST, SW52 SW_SPST, SW53 SW_SPST, SW54 SW_SPST, SW55 SW_SPST, SW56 SW_SPST, SW57 SW_SPST, SW58 SW_SPST, SW59 SW_SPST, SW6 SW_SPST, SW60 SW_SPST, SW61 SW_SPST, SW7 SW_SPST, SW8 SW_SPST, SW9 SW_SPST, U1 ATmega32U4-AU, X1 FA-238

Commit message: footprints, key arrangement, board dimensions
Parts:
- SW1, SW11, SW12, SW13, SW14, SW16, SW17, SW18, SW19, SW21, SW22, SW23, SW24, SW26, SW27, SW28, SW29, SW31, SW32, SW33, SW34, SW36, SW37, SW38, SW39, SW41, SW42, SW43, SW44, SW45, SW46, SW47, SW48, SW49, SW50, SW51, SW52, SW53, SW54, SW55, SW57, SW58, SW6, SW7, SW8, SW9: footprint 61key:SW_MX -> 61key:MX-1U-NoLED
- SW10, SW15, SW25, SW30, SW35, SW40, SW5: footprint 61key:SW_MX -> 61key:MX-1.25U-NoLED
- SW2, SW61: footprint 61key:SW_MX -> 61key:MX-1.5U-NoLED
- SW20: footprint 61key:SW_MX -> 61key:MX-6.25U-NoLED
- SW3: footprint 61key:SW_MX -> 61key:MX-1.75U-NoLED
- SW4, SW59: footprint 61key:SW_MX -> 61key:MX-2.25U-NoLED
- SW56: footprint 61key:SW_MX -> 61key:MX-2.75U-NoLED
- SW60: footprint 61key:SW_MX -> 61key:MX-2U-NoLED
- moved D59 306.8 mm to (-81.0, 107.2)
- moved D52 298.4 mm to (-66.7, 123.8)
- moved C2 298.0 mm to (-64.6, 112.3)
- moved D10 298.0 mm to (-95.5, 142.5)
- moved D11 298.0 mm to (-102.1, 125.5)
- moved D12 298.0 mm to (-87.6, 109.1)
- moved D13 298.0 mm to (-87.6, 113.4)
- moved D2 298.0 mm to (-79.3, 130.4)
- moved D23 298.0 mm to (-90.7, 130.4)
- moved D26 298.0 mm to (-79.3, 121.9)
- moved D29 298.0 mm to (-100.3, 151.9)
- moved D30 298.0 mm to (-95.5, 138.3)
- moved D31 298.0 mm to (-95.5, 146.8)
- moved D34 298.0 mm to (-102.1, 129.8)
- moved D36 298.0 mm to (-74.6, 104.9)
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Routing:
- net /row4: track 0.00 -> 261.9 mm
- net /row1: track 0.00 -> 257.2 mm
- net /row0: track 0.00 -> 257.2 mm
- net /row2: track 0.00 -> 247.7 mm
- net /row3: track 0.00 -> 238.1 mm
Other:
- board outline added: 295.3 x 100 mm
- net class Default: trace_width 0.25 -> 0.4

Commit message: basic pcb, issues with holes
Parts:
- added REF**: MountingHole_2.2mm_M2_DIN965_Pad, MountingHole:MountingHole_2.2mm_M2_DIN965_Pad, F.Cu at (200.0, 61.9)
- added REF**: MountingHole_2.2mm_M2_DIN965_Pad, MountingHole:MountingHole_2.2mm_M2_DIN965_Pad, F.Cu at (142.9, 61.9)
- added REF**: MountingHole_2.2mm_M2_DIN965_Pad, MountingHole:MountingHole_2.2mm_M2_DIN965_Pad, F.Cu at (181.0, 147.6)
- added REF**: MountingHole_2.2mm_M2_DIN965_Pad, MountingHole:MountingHole_2.2mm_M2_DIN965_Pad, F.Cu at (76.2, 81.0)
- added REF**: MountingHole_2.2mm_M2_DIN965_Pad, MountingHole:MountingHole_2.2mm_M2_DIN965_Pad, F.Cu at (266.7, 81.0)
- added REF**: MountingHole_2.2mm_M2_Pad_Via, MountingHole:MountingHole_2.2mm_M2_Pad_Via, F.Cu at (28.6, 61.9)
- added REF**: MountingHole_2.2mm_M2_Pad_Via, MountingHole:MountingHole_2.2mm_M2_Pad_Via, F.Cu at (28.6, 157.2)
- added REF**: MountingHole_2.2mm_M2_Pad_Via, MountingHole:MountingHole_2.2mm_M2_Pad_Via, F.Cu at (314.3, 157.2)
- added REF**: MountingHole_2.2mm_M2_Pad_Via, MountingHole:MountingHole_2.2mm_M2_Pad_Via, F.Cu at (314.3, 61.9)
- C1, C2, C3, J1, R1, R2, R3, R4, R5, R6, X1: moved to B.Cu
- D1, D10, D11, D12, D13, D14, D15, D16, D17, D18, D19, D2, D20, D21, D22, D23, D24, D25, D26, D27, D28, D29, D3, D30, D31, D32, D33, D34, D35, D36, D37, D38, D39, D4, D40, D41, D42, D43, D44, D45, D46, D47, D48, D49, D5, D50, D51, D52, D53, D54, D55, D56, D57, D58, D59, D6, D60, D61, D7, D8, D9: footprint Diode_THT:D_DO-41_SOD81_P7.62mm_Horizontal -> Diode_SMD:D_0805_2012Metric; moved to B.Cu
- U1: footprint Package_QFP:TQFP-44_10x10mm_P0.8mm -> 61key:QFN-44-1EP_7x7mm_Pitch0.5mm; moved to B.Cu
- moved D40 467.3 mm to (309.6, 142.6), turned to 180 degrees
- moved D35 454.8 mm to (285.8, 142.6), turned to 180 degrees
- moved D57 449.3 mm to (273.8, 66.4), turned to 180 degrees
- moved D55 439.4 mm to (269.1, 104.5), turned to 180 degrees
- moved D54 418.8 mm to (264.3, 85.4), turned to 180 degrees
- moved D60 410.1 mm to (302.4, 66.4), turned to 180 degrees
- moved D46 400.6 mm to (226.2, 85.4), turned to 180 degrees
- moved D53 393.5 mm to (254.8, 66.4), turned to 180 degrees
- moved D49 393.2 mm to (235.7, 66.4), turned to 180 degrees
- moved D25 384.5 mm to (238.1, 142.6), turned to 180 degrees
- moved D50 382.8 mm to (245.3, 85.4), turned to 180 degrees
- moved D56 374.7 mm to (272.7, 123.8)
- moved D51 370.8 mm to (250.0, 104.5), turned to 180 degrees
- moved D58 369.6 mm to (283.4, 85.4), turned to 180 degrees
- moved D59 367.9 mm to (286.9, 103.0)
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Connections:
- D20 pad 1: /col3 -> /col5
- D25 pad 1: /col4 -> /col9
- D30 pad 1: /col5 -> /col10
- D35 pad 1: /col6 -> /col11
- D40 pad 1: /col7 -> /col13
- D41 pad 1: /col7 -> /col8
- D42 pad 1: /col7 -> /col8
- D43 pad 1: /col7 -> /col8
- D44 pad 1: /col7 -> /col8
- D45 pad 1: /col8 -> /col9
- D46 pad 1: /col8 -> /col9
- D47 pad 1: /col8 -> /col9
- D48 pad 1: /col8 -> /col9
- D49 pad 1: /col9 -> /col10
- D50 pad 1: /col9 -> /col10
- D51 pad 1: /col9 -> /col10
- D52 pad 1: /col9 -> /col10
- D53 pad 1: /col10 -> /col11
- D54 pad 1: /col10 -> /col11
- D55 pad 1: /col10 -> /col11
- D56 pad 1: /col10 -> /col11
- D57 pad 1: Net-(D57-Pad1) -> /col12
- D58 pad 1: Net-(D57-Pad1) -> /col12
- D59 pad 1: Net-(D57-Pad1) -> /col12
- D60 pad 1: /col12 -> /col13
- D61 pad 1: /col12 -> /col13
- J1 pad A1: Net-(J1-PadA1) -> GND
- J1 pad A12: Net-(J1-PadA1) -> GND
- J1 pad B1: Net-(J1-PadA1) -> GND
- J1 pad B12: Net-(J1-PadA1) -> GND
- J1 pad S1: Net-(J1-PadA1) -> GND
- J1 pad S2: Net-(J1-PadA1) -> GND
- J1 pad S3: Net-(J1-PadA1) -> GND
- J1 pad S4: Net-(J1-PadA1) -> GND
- U1 pad 12: /col0 -> Net-(U1-Pad12)
- U1 pad 15: Net-(J1-PadA1) -> GND
- U1 pad 18: /col1 -> /col13
- U1 pad 19: /col2 -> /col12
- U1 pad 20: /col3 -> /col11
- U1 pad 21: /col4 -> /col10
- U1 pad 22: /col5 -> /col9
- U1 pad 23: Net-(J1-PadA1) -> GND
- U1 pad 25: Net-(U1-Pad25) -> /col7
- U1 pad 26: /row4 -> /col8
- U1 pad 27: /row3 -> /row4
- U1 pad 28: /row2 -> /row3
- U1 pad 29: /row1 -> /row2
- U1 pad 30: /row0 -> /row1
- U1 pad 31: Net-(U1-Pad31) -> /row0
- U1 pad 35: Net-(J1-PadA1) -> GND
- U1 pad 36: /col7 -> /col5
- U1 pad 37: /col8 -> /col4
- U1 pad 38: /col9 -> /col3
- U1 pad 39: /col10 -> /col2
- U1 pad 40: /col11 -> /col1
- U1 pad 41: /col12 -> /col0
- U1 pad 43: Net-(J1-PadA1) -> GND
- U1 pad 5: Net-(J1-PadA1) -> GND
Routing:
- net /col0: track 0.00 -> 221.6 mm, vias 0 -> 2
- net /col13: track 0.00 -> 206.9 mm, vias 0 -> 2
- net /col1: track 0.00 -> 193.0 mm, vias 0 -> 2
- net /col2: track 0.00 -> 178.8 mm, vias 0 -> 2
- net /col11: track 0.00 -> 172.4 mm, vias 0 -> 2
- net /col10: track 0.00 -> 151.2 mm, vias 0 -> 2
- net /col12: track 0.00 -> 143.9 mm, vias 0 -> 2
- net /col3: track 0.00 -> 135.0 mm, vias 0 -> 2
- net /col9: track 0.00 -> 132.0 mm, vias 0 -> 2
- net /col5: track 0.00 -> 116.6 mm, vias 0 -> 2
- net /col4: track 0.00 -> 115.7 mm, vias 0 -> 2
- net /col8: track 0.00 -> 95.9 mm, vias 0 -> 2
- net /row4: track 261.9 -> 354.4 mm
- net /col6: track 0.00 -> 78.8 mm, vias 0 -> 2
- net /col7: track 0.00 -> 72.4 mm, vias 0 -> 2
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- added copper zone on B.Cu, net GND
- added copper zone on F.Cu, net GND
Other:
- board size 295.3 x 100 mm -> 295.3 x 104.8 mm

Commit message: optimize entire board
Parts:
- removed the REF** at (200.0, 61.9)
- removed the REF** at (142.9, 61.9)
- added REF**: MountingHole_2.2mm_M2_DIN965_Pad, MountingHole:MountingHole_2.2mm_M2_DIN965_Pad, F.Cu at (242.9, 119.1)
- added REF**: MountingHole_2.2mm_M2_DIN965_Pad, MountingHole:MountingHole_2.2mm_M2_DIN965_Pad, F.Cu at (161.9, 81.0)
- added REF**: MountingHole_2.2mm_M2_DIN965_Pad, MountingHole:MountingHole_2.2mm_M2_DIN965_Pad, F.Cu at (100.0, 119.1)
- moved C2 20.9 mm to (190.8, 85.0), turned to 0 degrees
- moved D37 9.07 mm to (184.1, 93.8), turned to 90 degrees
- moved C3 4.38 mm to (194.8, 78.7)
- moved X1 3.91 mm to (190.7, 79.8)
- moved C1 3.61 mm to (190.8, 82.8)
- moved R4 3.19 mm to (179.8, 70.4)
- moved R3 2.34 mm to (182.1, 68.4)
- moved R6 2.08 mm to (176.3, 83.7), turned to 90 degrees
- moved R5 1.77 mm to (189.2, 75.0)
- moved U1 1.01 mm to (182.0, 78.0)
- moved D36 0.81 mm to (174.6, 75.6)
- moved R2 0.37 mm to (189.3, 61.9)
Connections:
- U1 pad 12: Net-(U1-Pad12) -> /col13
- U1 pad 18: /col13 -> /col12
- U1 pad 19: /col12 -> /col11
- U1 pad 20: /col11 -> /col10
- U1 pad 21: /col10 -> /col9
- U1 pad 22: /col9 -> /col8
- U1 pad 25: /col7 -> Net-(U1-Pad25)
- U1 pad 26: /col8 -> Net-(U1-Pad26)
- U1 pad 27: /row4 -> Net-(U1-Pad27)
- U1 pad 28: /row3 -> /row4
- U1 pad 29: /row2 -> /row3
- U1 pad 30: /row1 -> /row2
- U1 pad 31: /row0 -> /row1
- U1 pad 36: /col5 -> /col4
- U1 pad 37: /col4 -> /col3
- U1 pad 38: /col3 -> /col2
- U1 pad 39: /col2 -> /col1
- U1 pad 40: /col1 -> /col0
- U1 pad 41: /col0 -> /col7
- U1 pad 8: Net-(U1-Pad8) -> /row0
Routing:
- net /col5: track 116.6 -> 87.5 mm, vias 2 -> 0
- net /row0: track 279.5 -> 266.7 mm, vias 1 -> 0
- net Net-(C2-Pad1): track 8.53 -> 21.1 mm
- net /col12: track 143.9 -> 132.6 mm
- net /col8: track 95.9 -> 85.1 mm
- net /col11: track 172.4 -> 161.8 mm, vias 2 -> 3
- net /col10: track 151.2 -> 141.7 mm
- net /col9: track 132.0 -> 123.6 mm, vias 2 -> 3
- net Net-(J1-PadA7): track 3.75 -> 10.3 mm, vias 0 -> 3
- net /row4: track 354.4 -> 348.0 mm, vias 0 -> 1
- net Net-(J1-PadA6): track 10.2 -> 4.41 mm, vias 2 -> 0
- net /col7: track 72.4 -> 68.0 mm
- net /col4: track 115.7 -> 119.6 mm
- net Net-(C3-Pad2): track 13.0 -> 9.53 mm
- net /col3: track 135.0 -> 138.4 mm
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