File: 61key.sch (KiCad schematic (older format))
At the start: 134 parts, among them J1 105450-0101, SW1 SW_SPST, SW10 SW_SPST, SW11 SW_SPST, SW12 SW_SPST, SW13 SW_SPST, SW14 SW_SPST, SW15 SW_SPST, SW16 SW_SPST, SW17 SW_SPST, SW18 SW_SPST, SW19 SW_SPST, SW2 SW_SPST, SW20 SW_SPST, SW21 SW_SPST, SW22 SW_SPST, SW23 SW_SPST, SW24 SW_SPST, SW25 SW_SPST, SW26 SW_SPST, SW27 SW_SPST, SW28 SW_SPST, SW29 SW_SPST, SW3 SW_SPST, SW30 SW_SPST, SW31 SW_SPST, SW32 SW_SPST, SW33 SW_SPST, SW34 SW_SPST, SW35 SW_SPST, SW36 SW_SPST, SW37 SW_SPST, SW38 SW_SPST, SW39 SW_SPST, SW4 SW_SPST, SW40 SW_SPST, SW41 SW_SPST, SW42 SW_SPST, SW43 SW_SPST, SW44 SW_SPST, SW45 SW_SPST, SW46 SW_SPST, SW47 SW_SPST, SW48 SW_SPST, SW49 SW_SPST, SW5 SW_SPST, SW50 SW_SPST, SW51 SW_SPST, SW52 SW_SPST, SW53 SW_SPST, SW54 SW_SPST, SW55 SW_SPST, SW56 SW_SPST, SW57 SW_SPST, SW58 SW_SPST, SW59 SW_SPST, SW6 SW_SPST, SW60 SW_SPST, SW61 SW_SPST, SW7 SW_SPST, SW8 SW_SPST, SW9 SW_SPST, U1 ATmega32U4-AU, X1 FA-238

Commit message: footprints, key arrangement, board dimensions
Parts:
- SW1, SW11, SW12, SW13, SW14, SW16, SW17, SW18, SW19, SW21, SW22, SW23, SW24, SW26, SW27, SW28, SW29, SW31, SW32, SW33, SW34, SW36, SW37, SW38, SW39, SW41, SW42, SW43, SW44, SW45, SW46, SW47, SW48, SW49, SW50, SW51, SW52, SW53, SW54, SW55, SW57, SW58, SW6, SW7, SW8, SW9: footprint 61key:SW_MX -> 61key:MX-1U-NoLED
- SW10, SW15, SW25, SW30, SW35, SW40, SW5: footprint 61key:SW_MX -> 61key:MX-1.25U-NoLED
- SW2, SW61: footprint 61key:SW_MX -> 61key:MX-1.5U-NoLED
- SW20: footprint 61key:SW_MX -> 61key:MX-6.25U-NoLED
- SW3: footprint 61key:SW_MX -> 61key:MX-1.75U-NoLED
- SW4, SW59: footprint 61key:SW_MX -> 61key:MX-2.25U-NoLED
- SW56: footprint 61key:SW_MX -> 61key:MX-2.75U-NoLED
- SW60: footprint 61key:SW_MX -> 61key:MX-2U-NoLED

Commit message: basic pcb, issues with holes
Parts:
- D1, D10, D11, D12, D13, D14, D15, D16, D17, D18, D19, D2, D20, D21, D22, D23, D24, D25, D26, D27, D28, D29, D3, D30, D31, D32, D33, D34, D35, D36, D37, D38, D39, D4, D40, D41, D42, D43, D44, D45, D46, D47, D48, D49, D5, D50, D51, D52, D53, D54, D55, D56, D57, D58, D59, D6, D60, D61, D7, D8, D9: footprint Diode_THT:D_DO-41_SOD81_P7.62mm_Horizontal -> Diode_SMD:D_0805_2012Metric
- U1: footprint Package_QFP:TQFP-44_10x10mm_P0.8mm -> 61key:QFN-44-1EP_7x7mm_Pitch0.5mm
Connections:
- net GND: now also J1.A1 (GND1), J1.A12 (GND2), J1.B1 (GND3), J1.B12 (GND4), J1.S1 (SHIELD), J1.S2 (SHIELD), J1.S3 (SHIELD), J1.S4 (SHIELD), U1.15 (GND), U1.23 (GND), U1.35 (GND), U1.43 (GND), U1.5 (UGND)
- net col0: now also U1.41 (PF0); no longer U1.12 (PB7)
- net col1: now also U1.40 (PF1); no longer U1.18 (PD0)
- net col10: now also D30.1 (K), D49.1 (K), D50.1 (K), D51.1 (K), D52.1 (K), U1.21 (PD3); no longer D53.1 (K), D54.1 (K), D55.1 (K), D56.1 (K), U1.39 (PF4)
- net col11: now also D35.1 (K), D53.1 (K), D54.1 (K), D55.1 (K), D56.1 (K), U1.20 (PD2); no longer U1.40 (PF1)
- net col12: now also D57.1 (K), D58.1 (K), D59.1 (K), U1.19 (PD1); no longer D60.1 (K), D61.1 (K), U1.41 (PF0)
- net col2: now also U1.39 (PF4); no longer U1.19 (PD1)
- net col3: now also U1.38 (PF5); no longer D20.1 (K), U1.20 (PD2)
- net col4: now also U1.37 (PF6); no longer D25.1 (K), U1.21 (PD3)
- net col5: now also D20.1 (K), U1.36 (PF7); no longer D30.1 (K), U1.22 (PD5)
- net col6: no longer D35.1 (K)
- net col7: now also U1.25 (PD4); no longer D40.1 (K), D41.1 (K), D42.1 (K), D43.1 (K), D44.1 (K), U1.36 (PF7)
- net col8: now also D41.1 (K), D42.1 (K), D43.1 (K), D44.1 (K), U1.26 (PD6); no longer D45.1 (K), D46.1 (K), D47.1 (K), D48.1 (K), U1.37 (PF6)
- net col9: now also D25.1 (K), D45.1 (K), D46.1 (K), D47.1 (K), D48.1 (K), U1.22 (PD5); no longer D49.1 (K), D50.1 (K), D51.1 (K), D52.1 (K), U1.38 (PF5)
- net row0: now also U1.31 (PC6); no longer U1.30 (PB6)
- net row1: now also U1.30 (PB6); no longer U1.29 (PB5)
- net row2: now also U1.29 (PB5); no longer U1.28 (PB4)
- net row3: now also U1.28 (PB4); no longer U1.27 (PD7)
- net row4: now also U1.27 (PD7); no longer U1.26 (PD6)
- new net col13: D40.1 (K), D60.1 (K), D61.1 (K), U1.18 (PD0)
Other:
- moved on the sheet: R1

Commit message: optimize entire board
Connections:
- net col0: now also U1.40 (PF1); no longer U1.41 (PF0)
- net col1: now also U1.39 (PF4); no longer U1.40 (PF1)
- net col10: now also U1.20 (PD2); no longer U1.21 (PD3)
- net col11: now also U1.19 (PD1); no longer U1.20 (PD2)
- net col12: now also U1.18 (PD0); no longer U1.19 (PD1)
- net col13: now also U1.12 (PB7); no longer U1.18 (PD0)
- net col2: now also U1.38 (PF5); no longer U1.39 (PF4)
- net col3: now also U1.37 (PF6); no longer U1.38 (PF5)
- net col4: now also U1.36 (PF7); no longer U1.37 (PF6)
- net col5: no longer U1.36 (PF7)
- net col7: now also U1.41 (PF0); no longer U1.25 (PD4)
- net col8: now also U1.22 (PD5); no longer U1.26 (PD6)
- net col9: now also U1.21 (PD3); no longer U1.22 (PD5)
- net row0: now also U1.8 (PB0); no longer U1.31 (PC6)
- net row1: now also U1.31 (PC6); no longer U1.30 (PB6)
- net row2: now also U1.30 (PB6); no longer U1.29 (PB5)
- net row3: now also U1.29 (PB5); no longer U1.28 (PB4)
- net row4: now also U1.28 (PB4); no longer U1.27 (PD7)
Changed lines of the file:
@@
 Wire Wire Line
 	1350 5050 1350 4850
-Text Label 5500 6750 0    50   ~ 0
-col1
-Text Label 5500 6850 0    50   ~ 0
+Text Label 5500 6950 0    50   ~ 0
 col2
-Text Label 5500 6950 0    50   ~ 0
+Text Label 5500 7050 0    50   ~ 0
 col3
-Text Label 5500 7050 0    50   ~ 0
+Text Label 5500 7150 0    50   ~ 0
 col4
-Text Label 5500 7150 0    50   ~ 0
+Text Label 5800 7150 0    50   ~ 0
 col5
 Text Label 5500 5250 0    50   ~ 0
 col6
+Text Label 5500 4250 0    50   ~ 0
+row0
+Text Label 5500 6750 0    50   ~ 0
+col0
+Text Label 5500 4950 0    50   ~ 0
+col13
+Text Label 5500 5450 0    50   ~ 0
+col12
+Text Label 5500 5550 0    50   ~ 0
+col11
+Text Label 5500 4850 0    50   ~ 0
+row2
+Text Label 5500 4750 0    50   ~ 0
+row3
 Text Label 5500 5150 0    50   ~ 0
-row0
-Text Label 5500 6650 0    50   ~ 0
-col0
-Text Label 5500 5450 0    50   ~ 0
-col13
-Text Label 5500 5550 0    50   ~ 0
-col12
+row1
 Text Label 5500 5650 0    50   ~ 0
-col11
-Text Label 5500 4750 0    50   ~ 0
-row2
-Text Label 5500 4650 0    50   ~ 0
-row3
-Text Label 5500 5850 0    50   ~ 0
-col7
-Text Label 5500 4850 0    50   ~ 0
-row1
-Text Label 5500 5750 0    50   ~ 0
 col10
-Text Label 5500 6050 0    50   ~ 0
+Text Label 5500 5950 0    50   ~ 0
 col8
 Connection ~ 6800 3400
@@
 	9000 3800 9000 3400
 Connection ~ 9000 3400
-Text Label 5500 6150 0    50   ~ 0
+Text Label 5500 4650 0    50   ~ 0
 row4
-Text Label 5500 5950 0    50   ~ 0
+Text Label 5500 5750 0    50   ~ 0
 col9
+Text Label 5500 6650 0    50   ~ 0
+col7
+Text Label 5500 6850 0    50   ~ 0
+col1
 $EndSCHEMATC
