File: board/61key.kicad_pcb (KiCad board)
At the start: 2 copper layers, 295.3 x 104.8 mm, 147 parts, among them SW1 SW_SPST, SW10 SW_SPST, SW11 SW_SPST, SW12 SW_SPST, SW13 SW_SPST, SW14 SW_SPST, SW15 SW_SPST, SW16 SW_SPST, SW17 SW_SPST, SW18 SW_SPST, SW19 SW_SPST, SW2 SW_SPST, SW20 SW_SPST, SW21 SW_SPST, SW22 SW_SPST, SW23 SW_SPST, SW24 SW_SPST, SW25 SW_SPST, SW26 SW_SPST, SW27 SW_SPST, SW28 SW_SPST, SW29 SW_SPST, SW3 SW_SPST, SW30 SW_SPST, SW31 SW_SPST, SW32 SW_SPST, SW33 SW_SPST, SW34 SW_SPST, SW35 SW_SPST, SW36 SW_SPST, SW37 SW_SPST, SW38 SW_SPST, SW39 SW_SPST, SW4 SW_SPST, SW40 SW_SPST, SW41 SW_SPST, SW42 SW_SPST, SW43 SW_SPST, SW44 SW_SPST, SW45 SW_SPST, SW46 SW_SPST, SW47 SW_SPST, SW48 SW_SPST, SW49 SW_SPST, SW5 SW_SPST, SW50 SW_SPST, SW51 SW_SPST, SW52 SW_SPST, SW53 SW_SPST, SW54 SW_SPST, SW55 SW_SPST, SW56 SW_SPST, SW57 SW_SPST, SW58 SW_SPST, SW59 SW_SPST, SW6 SW_SPST, SW60 SW_SPST, SW61 SW_SPST, SW62 SW_SPST, SW63 SW_SPST, SW64 SW_SPST, SW65 SW_SPST, SW66 SW_SPST, SW67 SW_SPST, SW68 SW_SPST, SW69 SW_SPST, SW7 SW_SPST, SW70 SW_SPST, SW71 SW_SPST, SW72 SW_SPST, SW73 SW_SPST, SW74 SW_SPST, SW75 SW_SPST, SW8 SW_SPST, SW9 SW_SPST

Commit message: basic pcb done
Parts:
- added C1: 0.1uF, Capacitor_SMD:C_0603_1608Metric, B.Cu at (181.6, 137.5)
- added C2: 4.7uF, Capacitor_SMD:C_0603_1608Metric, B.Cu at (179.8, 137.5)
- added C3: 0.1uF, Capacitor_SMD:C_0603_1608Metric, B.Cu at (176.2, 137.5)
- added C4: 0.1uF, Capacitor_SMD:C_0603_1608Metric, B.Cu at (178.0, 137.5)
- added IC1: STM32, 61key:QFP80P900X900X160-32N, B.Cu at (167.6, 135.7)
- added J1: Conn_ARM_JTAG_SWD_10, Connector_PinHeader_2.54mm:PinHeader_2x05_P2.54mm_Vertical, B.Cu at (178.9, 149.1)
- added R1: 5.1k, Resistor_SMD:R_0603_1608Metric, B.Cu at (173.2, 61.3)
- added R3: 1k, Resistor_SMD:R_0603_1608Metric, B.Cu at (159.5, 131.9)
- added R4: 1k, Resistor_SMD:R_0603_1608Metric, B.Cu at (159.5, 133.4)
- added R5: 1k, Resistor_SMD:R_0603_1608Metric, B.Cu at (166.1, 129.2)
- added R6: 1k, Resistor_SMD:R_0603_1608Metric, B.Cu at (164.3, 129.2)
- added R7: 1k, Resistor_SMD:R_0603_1608Metric, B.Cu at (165.5, 145.3)
- added U1: LD1117S33TR_SOT223, Package_TO_SOT_SMD:SOT-223-3_TabPin2, B.Cu at (185.7, 79.2)
- added USB1: 12401598E4#2A, 61key:HRO-TYPE-C-31-M-12, B.Cu at (167.3, 66.0)
- D1, D10, D11, D12, D13, D14, D15, D16, D17, D18, D19, D2, D20, D21, D22, D23, D24, D25, D26, D27, D28, D29, D3, D30, D31, D32, D33, D34, D35, D36, D37, D38, D39, D4, D40, D41, D42, D43, D44, D45, D46, D47, D48, D49, D5, D50, D51, D52, D53, D54, D55, D56, D57, D58, D59, D6, D60, D61, D62, D63, D64, D65, D7, D8, D9: footprint 61key:D_0805_2012Metric -> Diode_SMD:D_SOD-123F
- R2: value R_US -> 5.1k; footprint Resistor_SMD:R_0805_2012Metric -> Resistor_SMD:R_0603_1608Metric
- moved R2 28.0 mm to (161.3, 61.3), turned to 90 degrees
- moved D20 5.66 mm to (158.1, 140.8), turned to 180 degrees
- turned D1 to 0 degrees
- turned D10 to 0 degrees
- turned D11 to 0 degrees
- turned D12 to 180 degrees
- turned D13 to 180 degrees
- turned D14 to 180 degrees
- turned D15 to 180 degrees
- turned D16 to 0 degrees
- turned D17 to 180 degrees
- turned D18 to 180 degrees
- turned D19 to 180 degrees
- turned D2 to 0 degrees
- turned D21 to 0 degrees
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Connections:
- net Net-(SW14-Pad1) renamed /row3
- D1 pad 1: /col0 -> Net-(D1-Pad1)
- D1 pad 2: Net-(D1-Pad2) -> /col0
- D10 pad 1: /col1 -> Net-(D10-Pad1)
- D10 pad 2: Net-(D10-Pad2) -> /col1
- D11 pad 1: /col2 -> Net-(D11-Pad1)
- D11 pad 2: Net-(D11-Pad2) -> /col2
- D12 pad 1: /col2 -> Net-(D12-Pad1)
- D12 pad 2: Net-(D12-Pad2) -> /col2
- D13 pad 1: /col2 -> Net-(D13-Pad1)
- D13 pad 2: Net-(D13-Pad2) -> /col2
- D14 pad 1: /col3 -> Net-(D14-Pad1)
- D14 pad 2: Net-(D14-Pad2) -> /col3
- D15 pad 1: /col2 -> Net-(D15-Pad1)
- D15 pad 2: Net-(D15-Pad2) -> /col2
- D16 pad 1: /col3 -> Net-(D16-Pad1)
- D16 pad 2: Net-(D16-Pad2) -> /col3
- D17 pad 1: /col3 -> Net-(D17-Pad1)
- D17 pad 2: Net-(D17-Pad2) -> /col3
- D18 pad 1: /col3 -> Net-(D18-Pad1)
- D18 pad 2: Net-(D18-Pad2) -> /col3
- D19 pad 1: /col4 -> Net-(D19-Pad1)
- D19 pad 2: Net-(D19-Pad2) -> /col4
- D2 pad 1: /col0 -> Net-(D2-Pad1)
- D2 pad 2: Net-(D2-Pad2) -> /col0
- D20 pad 1: /col6 -> Net-(D20-Pad1)
- D20 pad 2: Net-(D20-Pad2) -> /col6
- D21 pad 1: /col4 -> Net-(D21-Pad1)
- D21 pad 2: Net-(D21-Pad2) -> /col4
- D22 pad 1: /col4 -> Net-(D22-Pad1)
- D22 pad 2: Net-(D22-Pad2) -> /col4
- D23 pad 1: /col4 -> Net-(D23-Pad1)
- D23 pad 2: Net-(D23-Pad2) -> /col4
- D24 pad 1: /col5 -> Net-(D24-Pad1)
- D24 pad 2: Net-(D24-Pad2) -> /col5
- D25 pad 1: /col9 -> Net-(D25-Pad1)
- D25 pad 2: Net-(D25-Pad2) -> /col9
- D26 pad 1: /col5 -> Net-(D26-Pad1)
- D26 pad 2: Net-(D26-Pad2) -> /col5
- D27 pad 1: /col5 -> Net-(D27-Pad1)
- D27 pad 2: Net-(D27-Pad2) -> /col5
- D28 pad 1: /col5 -> Net-(D28-Pad1)
- D28 pad 2: Net-(D28-Pad2) -> /col5
- D29 pad 1: /col6 -> Net-(D29-Pad1)
- D29 pad 2: Net-(D29-Pad2) -> /col6
- D3 pad 1: /col0 -> Net-(D3-Pad1)
- D3 pad 2: Net-(D3-Pad2) -> /col0
- D30 pad 1: /col10 -> Net-(D30-Pad1)
- D30 pad 2: Net-(D30-Pad2) -> /col10
- D31 pad 1: /col6 -> Net-(D31-Pad1)
- D31 pad 2: Net-(D31-Pad2) -> /col6
- D32 pad 1: /col6 -> Net-(D32-Pad1)
- D32 pad 2: Net-(D32-Pad2) -> /col6
- D33 pad 1: /col6 -> Net-(D33-Pad1)
- D33 pad 2: Net-(D33-Pad2) -> /col6
- D34 pad 1: /col7 -> Net-(D34-Pad1)
- D34 pad 2: Net-(D34-Pad2) -> /col7
- D35 pad 1: /col11 -> Net-(D35-Pad1)
- D35 pad 2: Net-(D35-Pad2) -> /col11
- D36 pad 1: /col7 -> Net-(D36-Pad1)
- D36 pad 2: Net-(D36-Pad2) -> /col7
- D37 pad 1: /col7 -> Net-(D37-Pad1)
- D37 pad 2: Net-(D37-Pad2) -> /col7
- D38 pad 1: /col7 -> Net-(D38-Pad1)
- D38 pad 2: Net-(D38-Pad2) -> /col7
- D39 pad 1: /col8 -> Net-(D39-Pad1)
- D39 pad 2: Net-(D39-Pad2) -> /col8
- D4 pad 1: /col0 -> Net-(D4-Pad1)
- D4 pad 2: Net-(D4-Pad2) -> /col0
- D40 pad 1: /col13 -> Net-(D40-Pad1)
- D40 pad 2: Net-(D40-Pad2) -> /col13
- D41 pad 1: /col8 -> Net-(D41-Pad1)
- D41 pad 2: Net-(D41-Pad2) -> /col8
- D42 pad 1: /col8 -> Net-(D42-Pad1)
- D42 pad 2: Net-(D42-Pad2) -> /col8
- D43 pad 1: /col8 -> Net-(D43-Pad1)
- D43 pad 2: Net-(D43-Pad2) -> /col8
- D44 pad 1: /col9 -> Net-(D44-Pad1)
- D44 pad 2: Net-(D44-Pad2) -> /col9
- D45 pad 1: /col9 -> Net-(D45-Pad1)
- D45 pad 2: Net-(D45-Pad2) -> /col9
- D46 pad 1: /col9 -> Net-(D46-Pad1)
- D46 pad 2: Net-(D46-Pad2) -> /col9
- D47 pad 1: /col9 -> Net-(D47-Pad1)
- D47 pad 2: Net-(D47-Pad2) -> /col9
- D48 pad 1: /col10 -> Net-(D48-Pad1)
- D48 pad 2: Net-(D48-Pad2) -> /col10
- D49 pad 1: /col10 -> Net-(D49-Pad1)
- D49 pad 2: Net-(D49-Pad2) -> /col10
- D5 pad 1: /col0 -> Net-(D5-Pad1)
- D5 pad 2: Net-(D5-Pad2) -> /col0
- D50 pad 1: /col10 -> Net-(D50-Pad1)
- D50 pad 2: Net-(D50-Pad2) -> /col10
- D51 pad 1: /col10 -> Net-(D51-Pad1)
- D51 pad 2: Net-(D51-Pad2) -> /col10
- D52 pad 1: /col11 -> Net-(D52-Pad1)
- D52 pad 2: Net-(D52-Pad2) -> /col11
- D53 pad 1: /col11 -> Net-(D53-Pad1)
- D53 pad 2: Net-(D53-Pad2) -> /col11
- D54 pad 1: /col11 -> Net-(D54-Pad1)
- D54 pad 2: Net-(D54-Pad2) -> /col11
- D55 pad 1: /col11 -> Net-(D55-Pad1)
- D55 pad 2: Net-(D55-Pad2) -> /col11
- D56 pad 1: /col14 -> Net-(D56-Pad1)
- D56 pad 2: Net-(D56-Pad2) -> /col14
- D57 pad 1: /col12 -> Net-(D57-Pad1)
- D57 pad 2: Net-(D57-Pad2) -> /col12
- D58 pad 1: /col12 -> Net-(D58-Pad1)
- D58 pad 2: Net-(D58-Pad2) -> /col12
- D59 pad 1: /col13 -> Net-(D59-Pad1)
- D59 pad 2: Net-(D59-Pad2) -> /col13
- D6 pad 1: /col1 -> Net-(D6-Pad1)
- D6 pad 2: Net-(D6-Pad2) -> /col1
- D60 pad 1: /col13 -> Net-(D60-Pad1)
- D60 pad 2: Net-(D60-Pad2) -> /col13
- D61 pad 1: /col13 -> Net-(D61-Pad1)
- D61 pad 2: Net-(D61-Pad2) -> /col13
- D62 pad 1: /col14 -> Net-(D62-Pad1)
- D62 pad 2: Net-(D62-Pad2) -> /col14
- D63 pad 1: /col1 -> Net-(D63-Pad1)
- D63 pad 2: Net-(D63-Pad2) -> /col1
- D64 pad 1: /col13 -> Net-(D64-Pad1)
- D64 pad 2: Net-(D64-Pad2) -> /col13
- D65 pad 1: /col14 -> Net-(D65-Pad1)
- D65 pad 2: Net-(D65-Pad2) -> /col14
- D7 pad 1: /col1 -> Net-(D7-Pad1)
- D7 pad 2: Net-(D7-Pad2) -> /col1
- D8 pad 1: /col1 -> Net-(D8-Pad1)
- D8 pad 2: Net-(D8-Pad2) -> /col1
- D9 pad 1: /col2 -> Net-(D9-Pad1)
- D9 pad 2: Net-(D9-Pad2) -> /col2
- R2 pad 1: Net-(J1-PadB5) -> GND
- R2 pad 2: GND -> Net-(R2-Pad2)
- SW1 pad 2: Net-(D1-Pad2) -> Net-(D1-Pad1)
- SW10 pad 2: Net-(D10-Pad2) -> Net-(D10-Pad1)
- SW11 pad 2: Net-(D11-Pad2) -> Net-(D11-Pad1)
- SW12 pad 2: Net-(D12-Pad2) -> Net-(D12-Pad1)
- SW13 pad 2: Net-(D13-Pad2) -> Net-(D13-Pad1)
- SW14 pad 2: Net-(D14-Pad2) -> Net-(D14-Pad1)
- SW15 pad 2: Net-(D15-Pad2) -> Net-(D15-Pad1)
- SW16 pad 2: Net-(D16-Pad2) -> Net-(D16-Pad1)
- SW17 pad 2: Net-(D17-Pad2) -> Net-(D17-Pad1)
- SW18 pad 2: Net-(D18-Pad2) -> Net-(D18-Pad1)
- SW19 pad 2: Net-(D19-Pad2) -> Net-(D19-Pad1)
- SW2 pad 2: Net-(D2-Pad2) -> Net-(D2-Pad1)
- SW20 pad 2: Net-(D20-Pad2) -> Net-(D20-Pad1)
- SW21 pad 2: Net-(D21-Pad2) -> Net-(D21-Pad1)
- SW22 pad 2: Net-(D22-Pad2) -> Net-(D22-Pad1)
- SW23 pad 2: Net-(D23-Pad2) -> Net-(D23-Pad1)
- SW24 pad 2: Net-(D24-Pad2) -> Net-(D24-Pad1)
- SW25 pad 2: Net-(D25-Pad2) -> Net-(D25-Pad1)
- SW26 pad 2: Net-(D26-Pad2) -> Net-(D26-Pad1)
- SW27 pad 2: Net-(D27-Pad2) -> Net-(D27-Pad1)
- SW28 pad 2: Net-(D28-Pad2) -> Net-(D28-Pad1)
- SW29 pad 2: Net-(D29-Pad2) -> Net-(D29-Pad1)
- SW3 pad 2: Net-(D3-Pad2) -> Net-(D3-Pad1)
- SW30 pad 2: Net-(D30-Pad2) -> Net-(D30-Pad1)
- SW31 pad 2: Net-(D31-Pad2) -> Net-(D31-Pad1)
- SW32 pad 2: Net-(D32-Pad2) -> Net-(D32-Pad1)
- SW33 pad 2: Net-(D33-Pad2) -> Net-(D33-Pad1)
- SW34 pad 2: Net-(D34-Pad2) -> Net-(D34-Pad1)
- SW35 pad 2: Net-(D35-Pad2) -> Net-(D35-Pad1)
- SW36 pad 2: Net-(D36-Pad2) -> Net-(D36-Pad1)
- SW37 pad 2: Net-(D37-Pad2) -> Net-(D37-Pad1)
- SW38 pad 2: Net-(D38-Pad2) -> Net-(D38-Pad1)
- SW39 pad 2: Net-(D39-Pad2) -> Net-(D39-Pad1)
- SW4 pad 2: Net-(D4-Pad2) -> Net-(D4-Pad1)
- SW40 pad 2: Net-(D56-Pad2) -> Net-(D56-Pad1)
- SW41 pad 2: Net-(D41-Pad2) -> Net-(D41-Pad1)
- SW42 pad 2: Net-(D42-Pad2) -> Net-(D42-Pad1)
- SW43 pad 2: Net-(D43-Pad2) -> Net-(D43-Pad1)
- SW44 pad 2: Net-(D44-Pad2) -> Net-(D44-Pad1)
- SW45 pad 2: Net-(D45-Pad2) -> Net-(D45-Pad1)
- SW46 pad 2: Net-(D46-Pad2) -> Net-(D46-Pad1)
- SW47 pad 2: Net-(D47-Pad2) -> Net-(D47-Pad1)
- SW48 pad 2: Net-(D48-Pad2) -> Net-(D48-Pad1)
- SW49 pad 2: Net-(D49-Pad2) -> Net-(D49-Pad1)
- SW5 pad 2: Net-(D5-Pad2) -> Net-(D5-Pad1)
- SW50 pad 2: Net-(D50-Pad2) -> Net-(D50-Pad1)
- SW51 pad 2: Net-(D51-Pad2) -> Net-(D51-Pad1)
- SW52 pad 2: Net-(D52-Pad2) -> Net-(D52-Pad1)
- SW53 pad 2: Net-(D53-Pad2) -> Net-(D53-Pad1)
- SW54 pad 2: Net-(D54-Pad2) -> Net-(D54-Pad1)
- SW55 pad 2: Net-(D55-Pad2) -> Net-(D55-Pad1)
- SW56 pad 2: Net-(D64-Pad2) -> Net-(D64-Pad1)
- SW57 pad 2: Net-(D57-Pad2) -> Net-(D57-Pad1)
- SW58 pad 2: Net-(D58-Pad2) -> Net-(D58-Pad1)
- SW59 pad 2: Net-(D59-Pad2) -> Net-(D59-Pad1)
- SW6 pad 2: Net-(D6-Pad2) -> Net-(D6-Pad1)
- SW60 pad 2: Net-(D60-Pad2) -> Net-(D60-Pad1)
- SW61 pad 2: Net-(D61-Pad2) -> Net-(D61-Pad1)
- SW62 pad 2: Net-(D62-Pad2) -> Net-(D62-Pad1)
- SW63 pad 2: Net-(D60-Pad2) -> Net-(D60-Pad1)
- SW64 pad 2: Net-(D4-Pad2) -> Net-(D4-Pad1)
- SW65 pad 2: Net-(D63-Pad2) -> Net-(D63-Pad1)
- SW66 pad 2: Net-(D52-Pad2) -> Net-(D52-Pad1)
- SW67 pad 2: Net-(D64-Pad2) -> Net-(D64-Pad1)
- SW68 pad 2: Net-(D65-Pad2) -> Net-(D65-Pad1)
- SW69 pad 2: Net-(D25-Pad2) -> Net-(D25-Pad1)
- SW7 pad 2: Net-(D7-Pad2) -> Net-(D7-Pad1)
- SW70 pad 2: Net-(D30-Pad2) -> Net-(D30-Pad1)
- SW71 pad 2: Net-(D35-Pad2) -> Net-(D35-Pad1)
- SW72 pad 2: Net-(D40-Pad2) -> Net-(D40-Pad1)
- SW73 pad 2: Net-(D56-Pad2) -> Net-(D56-Pad1)
- SW74 pad 2: Net-(D59-Pad2) -> Net-(D59-Pad1)
- SW75 pad 2: Net-(D61-Pad2) -> Net-(D61-Pad1)
- SW8 pad 2: Net-(D8-Pad2) -> Net-(D8-Pad1)
- SW9 pad 2: Net-(D9-Pad2) -> Net-(D9-Pad1)
Routing:
- net /col12: track 19.6 -> 168.4 mm, vias 0 -> 2
- net /col14: track 76.5 -> 219.2 mm, vias 0 -> 2
- net /col13: track 92.2 -> 219.3 mm, vias 0 -> 2
- net /col0: track 85.1 -> 208.5 mm, vias 0 -> 2
- net +3V3: track 0.00 -> 108.9 mm
- net /col11: track 91.1 -> 193.3 mm, vias 0 -> 2
- net /col1: track 84.7 -> 183.3 mm, vias 0 -> 2
- net /col2: track 84.9 -> 166.3 mm, vias 0 -> 2
- net /D+: track 0.00 -> 76.6 mm
- net /D-: track 0.00 -> 76.4 mm
- net /col10: track 84.7 -> 161.0 mm, vias 0 -> 2
- net /row0: track 267.6 -> 342.5 mm
- net /col3: track 63.4 -> 137.9 mm
- net /row1: track 272.2 -> 332.5 mm
- net /col9: track 84.4 -> 141.8 mm, vias 0 -> 2
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Other:
- board text added: "GND"
- board text added: "RESET"
- board text added: "SWCLK"
- board text added: "SWDIO"
- board text added: "VCC"
- board text removed: "J1"

Commit message: need to create models to check board compatibility; prototype candidate
Parts:
- added C5: 4.7uF, Capacitor_SMD:C_0603_1608Metric, B.Cu at (186.1, 133.1)
- added J2: Conn_01x04_Female, 61key:exp_header, F.Cu at (312.5, 113.0)
- added J3: Conn_01x04_Female, 61key:exp_header, F.Cu at (298.8, 63.7)
- added J4: Conn_01x04_Female, 61key:exp_header, F.Cu at (30.4, 106.1)
- added J5: Conn_01x01_Female, TestPoint:TestPoint_Pad_4.0x4.0mm, B.Cu at (179.2, 158.7)
- added J6: Conn_01x01_Female, TestPoint:TestPoint_Pad_4.0x4.0mm, B.Cu at (173.8, 158.7)
- added R8: 4.7k, Resistor_SMD:R_0603_1608Metric, B.Cu at (186.3, 141.1)
- added R9: 4.7k, Resistor_SMD:R_0603_1608Metric, B.Cu at (184.5, 141.1)
- added REF**: 440_mounting_hole, 61key:440_mounting_hole, F.Cu at (314.3, 157.2)
- added REF**: 440_mounting_hole, 61key:440_mounting_hole, F.Cu at (314.3, 61.9)
- added REF**: 440_mounting_hole, 61key:440_mounting_hole, F.Cu at (28.6, 61.9)
- added REF**: 440_mounting_hole, 61key:440_mounting_hole, F.Cu at (28.6, 157.2)
- added REF**: 440_mounting_hole, 61key:440_mounting_hole, F.Cu at (104.8, 80.4)
- added REF**: 440_mounting_hole, 61key:440_mounting_hole, F.Cu at (238.1, 80.4)
- added REF**: 440_mounting_hole, 61key:440_mounting_hole, F.Cu at (126.2, 141.4)
- added REF**: 440_mounting_hole, 61key:440_mounting_hole, F.Cu at (216.7, 141.4)
- added REF**: 440_mounting_hole, 61key:440_mounting_hole, F.Cu at (171.5, 99.4)
- D1, D10, D11, D12, D13, D14, D15, D16, D17, D18, D19, D2, D20, D21, D22, D23, D24, D25, D26, D27, D28, D29, D3, D30, D31, D32, D33, D34, D35, D36, D37, D38, D39, D4, D40, D41, D42, D43, D44, D45, D46, D47, D48, D49, D5, D50, D51, D52, D53, D54, D55, D56, D57, D58, D59, D6, D60, D61, D62, D63, D64, D65, D7, D8, D9: footprint Diode_SMD:D_SOD-123F -> 61key:D_SOD-123F
- IC1: value STM32 -> STM32F042K6T6
- moved D60 12.2 mm to (298.2, 75.4), turned to 270 degrees
- moved USB1 9.74 mm to (167.3, 56.3), turned to 0 degrees
- moved D12 3.97 mm to (82.0, 85.4)
- moved D25 2.78 mm to (224.2, 140.4)
- moved D62 2.40 mm to (311.9, 66.4)
- moved R2 1.79 mm to (159.5, 61.3)
- moved R1 1.79 mm to (175.0, 61.3)
- moved R7 1.40 mm to (166.4, 144.2), turned to 90 degrees
- moved U1 1.06 mm to (185.7, 78.1), turned to 90 degrees
Connections:
- IC1 pad 20: /D+ -> /col7
- IC1 pad 22: /col7 -> /D+
- USB1 pad A5: Net-(R1-Pad2) -> Net-(R2-Pad2)
- USB1 pad B5: Net-(R2-Pad2) -> Net-(R1-Pad2)
Routing:
- net /SDA: track 0.00 -> 446.9 mm, vias 0 -> 4
- net /SCL: track 0.00 -> 439.6 mm, vias 0 -> 3
- net VBUS: track 28.5 -> 403.2 mm
- net /col14: track 219.2 -> 256.9 mm, vias 2 -> 3
- net /col13: track 219.3 -> 204.3 mm
- net +3V3: track 108.9 -> 120.5 mm, vias 0 -> 1
- net Net-(D12-Pad1): track 9.60 -> 4.89 mm
- net Net-(D60-Pad1): track 14.2 -> 17.5 mm
- net Net-(D25-Pad1): track 12.0 -> 8.75 mm
- net /D-: track 76.4 -> 78.8 mm
- net /col7: track 77.2 -> 79.2 mm, vias 0 -> 2
- net Net-(IC1-Pad6): track 5.31 -> 3.40 mm
- net Net-(R2-Pad2): track 6.56 -> 8.44 mm
- net /row4: track 278.2 -> 279.8 mm
- net /col9: track 141.8 -> 140.1 mm
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Other:
- board text added: "boot"
- board text added: "exp-a"
- board text added: "exp-b"
- board text added: "exp-c"
