File: board/61key.kicad_pcb (KiCad board)
At the start: 2 copper layers, 295.3 x 104.8 mm, 178 parts, among them IC1 STM32F042K6T6, J1 Conn_ARM_JTAG_SWD_10, J2 Conn_01x04_Female, J3 Conn_01x04_Female, J4 Conn_01x04_Female, J5 Conn_01x01_Female, J6 Conn_01x01_Female, SW1 SW_SPST, SW10 SW_SPST, SW11 SW_SPST, SW12 SW_SPST, SW13 SW_SPST, SW14 SW_SPST, SW15 SW_SPST, SW16 SW_SPST, SW17 SW_SPST, SW18 SW_SPST, SW19 SW_SPST, SW2 SW_SPST, SW20 SW_SPST, SW21 SW_SPST, SW22 SW_SPST, SW23 SW_SPST, SW24 SW_SPST, SW25 SW_SPST, SW26 SW_SPST, SW27 SW_SPST, SW28 SW_SPST, SW29 SW_SPST, SW3 SW_SPST, SW30 SW_SPST, SW31 SW_SPST, SW32 SW_SPST, SW33 SW_SPST, SW34 SW_SPST, SW35 SW_SPST, SW36 SW_SPST, SW37 SW_SPST, SW38 SW_SPST, SW39 SW_SPST, SW4 SW_SPST, SW40 SW_SPST, SW41 SW_SPST, SW42 SW_SPST, SW43 SW_SPST, SW44 SW_SPST, SW45 SW_SPST, SW46 SW_SPST, SW47 SW_SPST, SW48 SW_SPST, SW49 SW_SPST, SW5 SW_SPST, SW50 SW_SPST, SW51 SW_SPST, SW52 SW_SPST, SW53 SW_SPST, SW54 SW_SPST, SW55 SW_SPST, SW56 SW_SPST, SW57 SW_SPST, SW58 SW_SPST, SW59 SW_SPST, SW6 SW_SPST, SW60 SW_SPST, SW61 SW_SPST, SW62 SW_SPST, SW63 SW_SPST, SW64 SW_SPST, SW65 SW_SPST, SW66 SW_SPST, SW67 SW_SPST, SW68 SW_SPST, SW69 SW_SPST, SW7 SW_SPST, SW70 SW_SPST, SW71 SW_SPST, SW72 SW_SPST, SW73 SW_SPST, SW74 SW_SPST, SW75 SW_SPST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

Commit message: logos, gerber
Parts:
- added G***: LOGO, 61key:logo, F.Cu at (171.5, 109.5)

Commit message: cleanup
Parts:
- removed J5, J6: Conn_01x01_Female, TestPoint:TestPoint_Pad_4.0x4.0mm
- added REF**: Fiducial_1mm_Mask3mm, Fiducial:Fiducial_1mm_Mask3mm, B.Cu at (307.8, 157.2)
- added REF**: Fiducial_1mm_Mask3mm, Fiducial:Fiducial_1mm_Mask3mm, B.Cu at (28.6, 67.3)
- added REF**: Fiducial_1mm_Mask3mm, Fiducial:Fiducial_1mm_Mask3mm, B.Cu at (34.8, 154.2)
- added REF**: Fiducial_1mm_Mask2mm, Fiducial:Fiducial_1mm_Mask2mm, B.Cu at (172.0, 131.3)
- added REF**: Fiducial_1mm_Mask2mm, Fiducial:Fiducial_1mm_Mask2mm, B.Cu at (163.1, 140.2)
- added REF**: MountingHole_2.5mm, MountingHole:MountingHole_2.5mm, F.Cu at (158.9, 60.7)
- added REF**: MountingHole_2.5mm, MountingHole:MountingHole_2.5mm, F.Cu at (175.6, 60.7)
- J3: value Conn_01x04_Female -> Conn_01x02_Female; footprint 61key:exp_header -> Connector_PinHeader_2.54mm:PinHeader_1x02_P2.54mm_Vertical; moved to B.Cu
- moved J3 138.6 mm to (188.3, 147.3), turned to 90 degrees
- moved R1 14.4 mm to (168.1, 74.0)
- moved R2 8.00 mm to (162.9, 68.6)
- moved D36 6.57 mm to (180.5, 70.6), turned to 270 degrees
- moved D62 5.10 mm to (313.4, 71.3), turned to 270 degrees
- moved D40 4.06 mm to (289.8, 137.9)
- moved D64 3.50 mm to (292.2, 119.8)
- moved R7 2.42 mm to (164.4, 145.5), turned to 0 degrees
- moved J2 1.79 mm to (314.3, 113.0)
- moved J4 1.79 mm to (28.6, 106.1)
Connections:
- J3 pad 1: GND -> /col14
- J3 pad 2: /SDA -> +3V3
Routing:
- net /SCL: track 439.6 -> 381.2 mm, vias 3 -> 2
- net /SDA: track 446.9 -> 391.1 mm, vias 4 -> 3
- net /col14: track 256.9 -> 236.9 mm
- net /col7: track 79.2 -> 71.3 mm
- net Net-(D62-Pad1): track 3.21 -> 7.52 mm
- net /col13: track 204.3 -> 200.3 mm
- net +3V3: track 120.5 -> 116.5 mm, vias 1 -> 0
- net Net-(D36-Pad1): track 4.52 -> 7.65 mm
- net Net-(R2-Pad2): track 8.44 -> 5.80 mm
- net Net-(IC1-Pad6): track 3.40 -> 6.04 mm
- net VBUS: track 403.2 -> 400.6 mm
- net /SWCLK: track 17.6 -> 20.2 mm
- net /row4: track 279.8 -> 277.4 mm
- net /col0: track 208.5 -> 210.6 mm, vias 2 -> 3
- net Net-(R1-Pad2): track 8.22 -> 10.1 mm
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Other:
- board text added: "ANSI /?"
- board text added: "akegata denki device one rev. 1"
- board text added: "space"
- board text removed: "exp-a"
- board text removed: "standard /?"
- board text removed: "standard shift"

Commit message: add readme
Parts:
- removed the REF** at (307.8, 157.2)
- removed the REF** at (28.6, 67.3)
- removed the REF** at (172.0, 131.3)
- removed the REF** at (163.1, 140.2)
- added F2: Fiducial_1mm_Mask2mm, Fiducial:Fiducial_1mm_Mask2mm, B.Cu at (163.1, 140.2)
- added F3: Fiducial_1mm_Mask2mm, Fiducial:Fiducial_1mm_Mask2mm, B.Cu at (172.0, 131.3)
- added F4: Fiducial_1mm_Mask3mm, Fiducial:Fiducial_1mm_Mask3mm, B.Cu at (307.8, 157.2)
- added F5: Fiducial_1mm_Mask3mm, Fiducial:Fiducial_1mm_Mask3mm, B.Cu at (28.6, 67.3)
- renumbered REF** to F1
