File: board/61key.sch (KiCad schematic (older format))
At the start: 163 parts, among them IC1 STM32F042K6T6, J1 Conn_ARM_JTAG_SWD_10, J2 Conn_01x04_Female, J3 Conn_01x04_Female, J4 Conn_01x04_Female, J5 Conn_01x01_Female, J6 Conn_01x01_Female, SW1 SW_SPST, SW10 SW_SPST, SW11 SW_SPST, SW12 SW_SPST, SW13 SW_SPST, SW14 SW_SPST, SW15 SW_SPST, SW16 SW_SPST, SW17 SW_SPST, SW18 SW_SPST, SW19 SW_SPST, SW2 SW_SPST, SW20 SW_SPST, SW21 SW_SPST, SW22 SW_SPST, SW23 SW_SPST, SW24 SW_SPST, SW25 SW_SPST, SW26 SW_SPST, SW27 SW_SPST, SW28 SW_SPST, SW29 SW_SPST, SW3 SW_SPST, SW30 SW_SPST, SW31 SW_SPST, SW32 SW_SPST, SW33 SW_SPST, SW34 SW_SPST, SW35 SW_SPST, SW36 SW_SPST, SW37 SW_SPST, SW38 SW_SPST, SW39 SW_SPST, SW4 SW_SPST, SW40 SW_SPST, SW41 SW_SPST, SW42 SW_SPST, SW43 SW_SPST, SW44 SW_SPST, SW45 SW_SPST, SW46 SW_SPST, SW47 SW_SPST, SW48 SW_SPST, SW49 SW_SPST, SW5 SW_SPST, SW50 SW_SPST, SW51 SW_SPST, SW52 SW_SPST, SW53 SW_SPST, SW54 SW_SPST, SW55 SW_SPST, SW56 SW_SPST, SW57 SW_SPST, SW58 SW_SPST, SW59 SW_SPST, SW6 SW_SPST, SW60 SW_SPST, SW61 SW_SPST, SW62 SW_SPST, SW63 SW_SPST, SW64 SW_SPST, SW65 SW_SPST, SW66 SW_SPST, SW67 SW_SPST, SW68 SW_SPST, SW69 SW_SPST, SW7 SW_SPST, SW70 SW_SPST, SW71 SW_SPST, SW72 SW_SPST, SW73 SW_SPST, SW74 SW_SPST, SW75 SW_SPST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

Commit message: cleanup
Parts:
- removed J3: Conn_01x04_Female, 61key:exp_header, symbol Connector:Conn_01x04_Female
- removed J5, J6: Conn_01x01_Female, TestPoint:TestPoint_Pad_4.0x4.0mm, symbol Connector:Conn_01x01_Female
- added J3: Conn_01x02_Female, Connector_PinHeader_2.54mm:PinHeader_1x02_P2.54mm_Vertical, symbol Connector:Conn_01x02_Female
Connections:
- net +3V3: now also J3.2 (Pin_2)
- net col14: now also J3.1 (Pin_1)
Changed lines of the file:
@@
 	3300 7250 3300 7350
 $Comp
-L power:GND #PWR?
+L power:GND #PWR0101
 U 1 1 5ED76D70
 P 3300 7350
-F 0 "#PWR?" H 3300 7100 50  0001 C CNN
+F 0 "#PWR0101" H 3300 7100 50  0001 C CNN
 F 1 "GND" V 3305 7222 50  0000 R CNN
 F 2 "" H 3300 7350 50  0001 C CNN
@@
 	3600 5850 3600 5950
 $Comp
-L power:GND #PWR?
+L power:GND #PWR0102
 U 1 1 5EDEDA53
 P 3900 5950
-F 0 "#PWR?" H 3900 5700 50  0001 C CNN
+F 0 "#PWR0102" H 3900 5700 50  0001 C CNN
 F 1 "GND" V 3905 5822 50  0000 R CNN
 F 2 "" H 3900 5950 50  0001 C CNN
@@
 $EndComp
 $Comp
-L power:GND #PWR?
+L power:GND #PWR0103
 U 1 1 5EDEE312
 P 3900 5650
-F 0 "#PWR?" H 3900 5400 50  0001 C CNN
+F 0 "#PWR0103" H 3900 5400 50  0001 C CNN
 F 1 "GND" V 3905 5522 50  0000 R CNN
 F 2 "" H 3900 5650 50  0001 C CNN
@@
 	2250 1050 2250 1150
 $Comp
-L power:GND #PWR?
+L power:GND #PWR0104
 U 1 1 5EE11FCF
 P 2250 1050
-F 0 "#PWR?" H 2250 800 50  0001 C CNN
+F 0 "#PWR0104" H 2250 800 50  0001 C CNN
 F 1 "GND" V 2255 922 50  0000 R CNN
 F 2 "" H 2250 1050 50  0001 C CNN
@@
 RESET
 $Comp
-L power:+3.3V #PWR?
+L power:+3.3V #PWR0105
 U 1 1 5EE21A11
 P 2100 4950
-F 0 "#PWR?" H 2100 4800 50  0001 C CNN
+F 0 "#PWR0105" H 2100 4800 50  0001 C CNN
 F 1 "+3.3V" V 2115 5078 50  0000 L CNN
 F 2 "" H 2100 4950 50  0001 C CNN
@@
 $EndComp
 $Comp
-L power:GND #PWR?
+L power:GND #PWR0106
 U 1 1 5EEA7ECB
 P 5100 6150
-F 0 "#PWR?" H 5100 5900 50  0001 C CNN
+F 0 "#PWR0106" H 5100 5900 50  0001 C CNN
 F 1 "GND" H 5105 5977 50  0000 C CNN
 F 2 "" H 5100 6150 50  0001 C CNN
@@
 $EndComp
 $Comp
-L power:VBUS #PWR?
+L power:VBUS #PWR0107
 U 1 1 5EEDEE31
 P 3300 6050
-F 0 "#PWR?" H 3300 5900 50  0001 C CNN
+F 0 "#PWR0107" H 3300 5900 50  0001 C CNN
 F 1 "VBUS" V 3315 6178 50  0000 L CNN
 F 2 "" H 3300 6050 50  0001 C CNN
@@
 Connection ~ 3300 6050
 $Comp
-L power:VBUS #PWR?
+L power:VBUS #PWR0108
 U 1 1 5EEEAF9A
 P 4800 5850
-F 0 "#PWR?" H 4800 5700 50  0001 C CNN
+F 0 "#PWR0108" H 4800 5700 50  0001 C CNN
 F 1 "VBUS" V 4815 5977 50  0000 L CNN
 F 2 "" H 4800 5850 50  0001 C CNN
@@
 $EndComp
 $Comp
-L power:GND #PWR?
+L power:GND #PWR0109
 U 1 1 5EEECC2C
 P 4250 7250
-F 0 "#PWR?" H 4250 7000 50  0001 C CNN
+F 0 "#PWR0109" H 4250 7000 50  0001 C CNN
 F 1 "GND" H 4255 7077 50  0000 C CNN
 F 2 "" H 4250 7250 50  0001 C CNN
@@
 	5400 5850 5500 5850
 $Comp
-L power:+3.3V #PWR?
+L power:+3.3V #PWR0110
 U 1 1 5EF73C5A
 P 5500 5850
-F 0 "#PWR?" H 5500 5700 50  0001 C CNN
+F 0 "#PWR0110" H 5500 5700 50  0001 C CNN
 F 1 "+3.3V" V 5515 5978 50  0000 L CNN
 F 2 "" H 5500 5850 50  0001 C CNN
@@
 Connection ~ 4700 7100
 $Comp
-L power:+3.3V #PWR?
+L power:+3.3V #PWR0111
 U 1 1 5F034C14
 P 4250 6650
-F 0 "#PWR?" H 4250 6500 50  0001 C CNN
+F 0 "#PWR0111" H 4250 6500 50  0001 C CNN
 F 1 "+3.3V" H 4265 6823 50  0000 C CNN
 F 2 "" H 4250 6650 50  0001 C CNN
@@
 	7150 6900 7250 6900
 $Comp
-L power:GND #PWR?
+L power:GND #PWR0112
 U 1 1 5F0DE9BE
 P 7250 6900
-F 0 "#PWR?" H 7250 6650 50  0001 C CNN
+F 0 "#PWR0112" H 7250 6650 50  0001 C CNN
 F 1 "GND" H 7255 6727 50  0000 C CNN
 F 2 "" H 7250 6900 50  0001 C CNN
@@
 Connection ~ 7250 6900
 $Comp
-L power:+3.3V #PWR?
+L power:+3.3V #PWR0113
 U 1 1 5F0E6759
 P 7250 5700
-F 0 "#PWR?" H 7250 5550 50  0001 C CNN
+F 0 "#PWR0113" H 7250 5550 50  0001 C CNN
 F 1 "+3.3V" H 7265 5873 50  0000 C CNN
 F 2 "" H 7250 5700 50  0001 C CNN
@@
 SCL
 $Comp
-L Connector:Conn_01x04_Female J3
-U 1 1 5ECA0E76
-P 9100 5700
-F 0 "J3" H 9128 5676 50  0000 L CNN
-F 1 "Conn_01x04_Female" H 9128 5585 50  0000 L CNN
-F 2 "61key:exp_header" H 9100 5700 50  0001 C CNN
-F 3 "~" H 9100 5700 50  0001 C CNN
-	1    9100 5700
-	1    0    0    -1
-$EndComp
-Text Label 8900 5600 2    50   ~ 0
-GND
-Text Label 8900 5700 2    50   ~ 0
-SDA
-Text Label 8900 5900 2    50   ~ 0
-SCL
-$Comp
 L Connector:Conn_01x04_Female J4
 U 1 1 5ECBAF65
@@
 SCL
 $Comp
-L power:VBUS #PWR?
+L power:VBUS #PWR0114
 U 1 1 5ED6E128
 P 8900 5350
-F 0 "#PWR?" H 8900 5200 50  0001 C CNN
+F 0 "#PWR0114" H 8900 5200 50  0001 C CNN
 F 1 "VBUS" V 8915 5477 50  0000 L CNN
 F 2 "" H 8900 5350 50  0001 C CNN
@@
 $EndComp
 $Comp
-L power:VBUS #PWR?
-U 1 1 5ED6FA6E
-P 8900 5800
-F 0 "#PWR?" H 8900 5650 50  0001 C CNN
-F 1 "VBUS" V 8915 5927 50  0000 L CNN
-F 2 "" H 8900 5800 50  0001 C CNN
-F 3 "" H 8900 5800 50  0001 C CNN
-	1    8900 5800
-	0    -1   -1   0
-$EndComp
-$Comp
-L power:VBUS #PWR?
+L power:VBUS #PWR0115
 U 1 1 5ED7AAFA
 P 8900 6300
-F 0 "#PWR?" H 8900 6150 50  0001 C CNN
+F 0 "#PWR0115" H 8900 6150 50  0001 C CNN
 F 1 "VBUS" V 8915 6427 50  0000 L CNN
 F 2 "" H 8900 6300 50  0001 C CNN
@@
 SDA
 $Comp
-L power:+3.3V #PWR?
+L power:+3.3V #PWR0116
 U 1 1 5EDFE690
 P 4350 5150
-F 0 "#PWR?" H 4350 5000 50  0001 C CNN
+F 0 "#PWR0116" H 4350 5000 50  0001 C CNN
 F 1 "+3.3V" V 4365 5278 50  0000 L CNN
 F 2 "" H 4350 5150 50  0001 C CNN
@@
 SCL
 $Comp
-L power:+3.3V #PWR?
+L power:+3.3V #PWR0117
 U 1 1 5EDFF2AF
 P 4350 5450
-F 0 "#PWR?" H 4350 5300 50  0001 C CNN
+F 0 "#PWR0117" H 4350 5300 50  0001 C CNN
 F 1 "+3.3V" V 4365 5578 50  0000 L CNN
 F 2 "" H 4350 5450 50  0001 C CNN
@@
 	0    1    1    0
 $EndComp
-$Comp
-L Connector:Conn_01x01_Female J5
-U 1 1 5EF11C5C
-P 1550 3100
-F 0 "J5" H 1578 3126 50  0000 L CNN
-F 1 "Conn_01x01_Female" H 1578 3035 50  0000 L CNN
-F 2 "TestPoint:TestPoint_Pad_4.0x4.0mm" H 1550 3100 50  0001 C CNN
-F 3 "~" H 1550 3100 50  0001 C CNN
-	1    1550 3100
-	1    0    0    -1
-$EndComp
-$Comp
-L Connector:Conn_01x01_Female J6
-U 1 1 5EF15230
-P 1550 3300
-F 0 "J6" H 1578 3326 50  0000 L CNN
-F 1 "Conn_01x01_Female" H 1578 3235 50  0000 L CNN
-F 2 "TestPoint:TestPoint_Pad_4.0x4.0mm" H 1550 3300 50  0001 C CNN
-F 3 "~" H 1550 3300 50  0001 C CNN
-	1    1550 3300
-	1    0    0    -1
-$EndComp
-Text Label 1350 3100 2    50   ~ 0
+Text Label 1300 2600 2    50   ~ 0
 col14
 $Comp
-L power:+3.3V #PWR?
+L power:+3.3V #PWR0118
 U 1 1 5EF2193C
-P 1350 3300
-F 0 "#PWR?" H 1350 3150 50  0001 C CNN
-F 1 "+3.3V" V 1365 3428 50  0000 L CNN
-F 2 "" H 1350 3300 50  0001 C CNN
-F 3 "" H 1350 3300 50  0001 C CNN
-	1    1350 3300
+P 1300 2700
+F 0 "#PWR0118" H 1300 2550 50  0001 C CNN
+F 1 "+3.3V" V 1315 2828 50  0000 L CNN
+F 2 "" H 1300 2700 50  0001 C CNN
+F 3 "" H 1300 2700 50  0001 C CNN
+	1    1300 2700
 	0    -1   -1   0
 $EndComp
@@
 	6150 6800 5650 6800
 Connection ~ 5650 6800
+$Comp
+L Connector:Conn_01x02_Female J3
+U 1 1 5ED5A495
+P 1500 2600
+F 0 "J3" H 1528 2576 50  0000 L CNN
+F 1 "Conn_01x02_Female" H 1528 2485 50  0000 L CNN
+F 2 "Connector_PinHeader_2.54mm:PinHeader_1x02_P2.54mm_Vertical" H 1500 2600 50  0001 C CNN
+F 3 "~" H 1500 2600 50  0001 C CNN
+	1    1500 2600
+	1    0    0    -1
+$EndComp
 $EndSCHEMATC
