File: backplate/backplate.kicad_pcb (KiCad board)
At the start: 2 copper layers, 295.3 x 104.8 mm, 4 parts

Commit message: need to create models to check board compatibility; prototype candidate
Parts:
- removed REF** (x4): MountingHole_2.2mm_M2_Pad_Via, MountingHole:MountingHole_2.2mm_M2_Pad_Via
- added J1: Conn_01x01_Male, backplate:sound_mounting_hole, F.Cu at (42.9, 61.9)
- added J2: Conn_01x01_Male, backplate:sound_mounting_hole, F.Cu at (42.9, 157.2)
- added J3: Conn_01x01_Male, backplate:sound_mounting_hole, F.Cu at (119.1, 80.4)
- added J4: Conn_01x01_Male, backplate:sound_mounting_hole, F.Cu at (185.7, 99.4)
- added J5: Conn_01x01_Male, backplate:sound_mounting_hole, F.Cu at (252.4, 80.4)
- added J6: Conn_01x01_Male, backplate:sound_mounting_hole, F.Cu at (140.5, 141.4)
- added J7: Conn_01x01_Male, backplate:sound_mounting_hole, F.Cu at (328.6, 61.9)
- added J8: Conn_01x01_Male, backplate:sound_mounting_hole, F.Cu at (328.6, 157.2)
- added J9: Conn_01x01_Male, backplate:sound_mounting_hole, F.Cu at (231.0, 141.4)
Routing:
- added copper zone on B.Cu, net GND
- added copper zone on F.Cu, net GND

Commit message: logos, gerber
Parts:
- added G***: LOGO, backplate:logo, F.Cu at (185.7, 109.5)

Commit message: cleanup
Other:
- board text added: "A"
- board text added: "B"
- board text added: "C"
- board text added: "D"
Changed lines of the file:
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@@
-(kicad_pcb (version 20171130) (host pcbnew 5.1.5)
+(kicad_pcb (version 20171130) (host pcbnew 5.1.6)
   (general
     (thickness 1.6)
-    (drawings 8)
+    (drawings 16)
     (tracks 0)
     (zones 0)
@@
     (38 B.Mask user hide)
     (39 F.Mask user hide)
-    (40 Dwgs.User user hide)
+    (40 Dwgs.User user)
     (41 Cmts.User user hide)
     (42 Eco1.User user)
@@
     (visible_elements FFFFFF7F)
     (pcbplotparams
-      (layerselection 0x010fc_ffffffff)
+      (layerselection 0x010f0_ffffffff)
       (usegerberextensions false)
       (usegerberattributes false)
@@
       (effects (font (size 1 1) (thickness 0.15)))
     )
-    (fp_text user %R (at 0.3 0) (layer F.Fab) hide
-      (effects (font (size 1 1) (thickness 0.15)))
-    )
-    (fp_circle (center 0 0) (end 3.5 0) (layer Cmts.User) (width 0.15))
-    (fp_circle (center 0 0) (end 3.75 0) (layer F.CrtYd) (width 0.05))
+    (fp_circle (center 0 0) (end 3.5 0) (layer Cmts.User) (width 0.15))
+    (fp_circle (center 0 0) (end 3.75 0) (layer F.CrtYd) (width 0.05))
+    (fp_text user %R (at 0.3 0) (layer F.Fab) hide
+      (effects (font (size 1 1) (thickness 0.15)))
+    )
     (pad 1 thru_hole circle (at 0 0) (size 5.5 5.5) (drill 3.5) (layers *.Cu *.Mask)
       (net 1 GND))
@@
       (effects (font (size 1 1) (thickness 0.15)))
     )
-    (fp_text user %R (at 0.3 0) (layer F.Fab) hide
-      (effects (font (size 1 1) (thickness 0.15)))
-    )
-    (fp_circle (center 0 0) (end 3.5 0) (layer Cmts.User) (width 0.15))
-    (fp_circle (center 0 0) (end 3.75 0) (layer F.CrtYd) (width 0.05))
+    (fp_circle (center 0 0) (end 3.5 0) (layer Cmts.User) (width 0.15))
+    (fp_circle (center 0 0) (end 3.75 0) (layer F.CrtYd) (width 0.05))
+    (fp_text user %R (at 0.3 0) (layer F.Fab) hide
+      (effects (font (size 1 1) (thickness 0.15)))
+    )
     (pad 1 thru_hole circle (at 0 0) (size 5.5 5.5) (drill 3.5) (layers *.Cu *.Mask)
       (net 1 GND))
@@
       (effects (font (size 1 1) (thickness 0.15)))
     )
-    (fp_text user %R (at 0.3 0) (layer F.Fab) hide
-      (effects (font (size 1 1) (thickness 0.15)))
-    )
-    (fp_circle (center 0 0) (end 3.5 0) (layer Cmts.User) (width 0.15))
-    (fp_circle (center 0 0) (end 3.75 0) (layer F.CrtYd) (width 0.05))
+    (fp_circle (center 0 0) (end 3.5 0) (layer Cmts.User) (width 0.15))
+    (fp_circle (center 0 0) (end 3.75 0) (layer F.CrtYd) (width 0.05))
+    (fp_text user %R (at 0.3 0) (layer F.Fab) hide
+      (effects (font (size 1 1) (thickness 0.15)))
+    )
     (pad 1 thru_hole circle (at 0 0) (size 5.5 5.5) (drill 3.5) (layers *.Cu *.Mask)
       (net 1 GND))
@@
       (effects (font (size 1 1) (thickness 0.15)))
     )
-    (fp_text user %R (at 0.3 0) (layer F.Fab) hide
-      (effects (font (size 1 1) (thickness 0.15)))
-    )
-    (fp_circle (center 0 0) (end 3.5 0) (layer Cmts.User) (width 0.15))
-    (fp_circle (center 0 0) (end 3.75 0) (layer F.CrtYd) (width 0.05))
+    (fp_circle (center 0 0) (end 3.5 0) (layer Cmts.User) (width 0.15))
+    (fp_circle (center 0 0) (end 3.75 0) (layer F.CrtYd) (width 0.05))
+    (fp_text user %R (at 0.3 0) (layer F.Fab) hide
+      (effects (font (size 1 1) (thickness 0.15)))
+    )
     (pad 1 thru_hole circle (at 0 0) (size 5.5 5.5) (drill 3.5) (layers *.Cu *.Mask)
       (net 1 GND))
@@
       (effects (font (size 1 1) (thickness 0.15)))
     )
-    (fp_text user %R (at 0.3 0) (layer F.Fab) hide
-      (effects (font (size 1 1) (thickness 0.15)))
-    )
-    (fp_circle (center 0 0) (end 3.5 0) (layer Cmts.User) (width 0.15))
-    (fp_circle (center 0 0) (end 3.75 0) (layer F.CrtYd) (width 0.05))
+    (fp_circle (center 0 0) (end 3.5 0) (layer Cmts.User) (width 0.15))
+    (fp_circle (center 0 0) (end 3.75 0) (layer F.CrtYd) (width 0.05))
+    (fp_text user %R (at 0.3 0) (layer F.Fab) hide
+      (effects (font (size 1 1) (thickness 0.15)))
+    )
     (pad 1 thru_hole circle (at 0 0) (size 5.5 5.5) (drill 3.5) (layers *.Cu *.Mask)
       (net 1 GND))
@@
       (effects (font (size 1 1) (thickness 0.15)))
     )
-    (fp_text user %R (at 0.3 0) (layer F.Fab) hide
-      (effects (font (size 1 1) (thickness 0.15)))
-    )
-    (fp_circle (center 0 0) (end 3.5 0) (layer Cmts.User) (width 0.15))
-    (fp_circle (center 0 0) (end 3.75 0) (layer F.CrtYd) (width 0.05))
+    (fp_circle (center 0 0) (end 3.5 0) (layer Cmts.User) (width 0.15))
+    (fp_circle (center 0 0) (end 3.75 0) (layer F.CrtYd) (width 0.05))
+    (fp_text user %R (at 0.3 0) (layer F.Fab) hide
+      (effects (font (size 1 1) (thickness 0.15)))
+    )
     (pad 1 thru_hole circle (at 0 0) (size 5.5 5.5) (drill 3.5) (layers *.Cu *.Mask)
       (net 1 GND))
@@
       (effects (font (size 1 1) (thickness 0.15)))
     )
-    (fp_text user %R (at 0.3 0) (layer F.Fab) hide
-      (effects (font (size 1 1) (thickness 0.15)))
-    )
-    (fp_circle (center 0 0) (end 3.5 0) (layer Cmts.User) (width 0.15))
-    (fp_circle (center 0 0) (end 3.75 0) (layer F.CrtYd) (width 0.05))
+    (fp_circle (center 0 0) (end 3.5 0) (layer Cmts.User) (width 0.15))
+    (fp_circle (center 0 0) (end 3.75 0) (layer F.CrtYd) (width 0.05))
+    (fp_text user %R (at 0.3 0) (layer F.Fab) hide
+      (effects (font (size 1 1) (thickness 0.15)))
+    )
     (pad 1 thru_hole circle (at 0 0) (size 5.5 5.5) (drill 3.5) (layers *.Cu *.Mask)
       (net 1 GND))
@@
       (effects (font (size 1 1) (thickness 0.15)))
     )
-    (fp_text user %R (at 0.3 0) (layer F.Fab) hide
-      (effects (font (size 1 1) (thickness 0.15)))
-    )
-    (fp_circle (center 0 0) (end 3.5 0) (layer Cmts.User) (width 0.15))
-    (fp_circle (center 0 0) (end 3.75 0) (layer F.CrtYd) (width 0.05))
-    (pad 1 thru_hole circle (at 0 0) (size 5.5 5.5) (drill 3.5) (layers *.Cu *.Mask)
-      (net 1 GND))
-  )
+    (fp_circle (center 0 0) (end 3.5 0) (layer Cmts.User) (width 0.15))
+    (fp_circle (center 0 0) (end 3.75 0) (layer F.CrtYd) (width 0.05))
+    (fp_text user %R (at 0.3 0) (layer F.Fab) hide
+      (effects (font (size 1 1) (thickness 0.15)))
+    )
+    (pad 1 thru_hole circle (at 0 0) (size 5.5 5.5) (drill 3.5) (layers *.Cu *.Mask)
+      (net 1 GND))
+  )
+  (gr_text D (at 323.850816 152.400384) (layer F.SilkS)
+    (effects (font (size 5 5) (thickness 0.75)))
+  )
+  (gr_text C (at 47.62512 152.400384) (layer F.SilkS)
+    (effects (font (size 5 5) (thickness 0.75)))
+  )
+  (gr_circle (center 333.37584 161.925408) (end 353.37584 161.925408) (layer Dwgs.User) (width 0.15))
+  (gr_circle (center 38.100096 161.925408) (end 58.100096 161.925408) (layer Dwgs.User) (width 0.15))
+  (gr_text B (at 323.850816 66.675168) (layer F.SilkS)
+    (effects (font (size 5 5) (thickness 0.75)))
+  )
+  (gr_circle (center 333.37584 57.150144) (end 353.37584 57.150144) (layer Dwgs.User) (width 0.15))
+  (gr_text A (at 47.62512 66.675168) (layer F.SilkS)
+    (effects (font (size 5 5) (thickness 0.75)))
+  )
+  (gr_circle (center 38.100096 57.150144) (end 58.100096 57.150144) (layer Dwgs.User) (width 0.15))
   (gr_arc (start 42.8625 61.9125) (end 42.8625 57.15) (angle -90) (layer Edge.Cuts) (width 0.05))
   (gr_arc (start 42.8625 157.1625) (end 38.1 157.1625) (angle -90) (layer Edge.Cuts) (width 0.05))
